File: cad/xmas-board/xmas-board.kicad_pcb (KiCad board)
At the start: 2 copper layers, 48.5 x 59.2 mm, 36 parts, among them J2 Pin Headers, SW1 KMR421NGLFS, SW3 On/Off Switch JS202011JCQN, U1 ATtiny25V-10S

Commit message: Update silkscreen and button position
Parts:
- moved SW1 0.40 mm to (67.3, 96.6)
Routing:
- net Net-(J2-Pin_2): track 42.2 -> 41.3 mm
Changed lines of the file:
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@@
 		(attr through_hole exclude_from_bom)
 		(fp_line
-			(start 3.92 -1.38)
-			(end 3.92 6.46)
-			(stroke
-				(width 0.12)
-				(type solid)
-			)
-			(layer "F.SilkS")
-		)
-		(fp_line
-			(start 1.27 -1.38)
-			(end 3.92 -1.38)
-			(stroke
-				(width 0.12)
-				(type solid)
-			)
-			(layer "F.SilkS")
-		)
-		(fp_line
-			(start -1.38 -1.38)
-			(end 0 -1.38)
-			(stroke
-				(width 0.12)
-				(type solid)
-			)
-			(layer "F.SilkS")
-		)
-		(fp_line
-			(start -1.38 0)
-			(end -1.38 -1.38)
-			(stroke
-				(width 0.12)
-				(type solid)
-			)
-			(layer "F.SilkS")
-		)
-		(fp_line
-			(start -1.38 1.27)
-			(end -1.38 6.46)
-			(stroke
-				(width 0.12)
-				(type solid)
-			)
-			(layer "F.SilkS")
-		)
-		(fp_line
-			(start -1.38 6.46)
-			(end 3.92 6.46)
-			(stroke
-				(width 0.12)
-				(type solid)
-			)
-			(layer "F.SilkS")
-		)
-		(fp_line
 			(start 4.32 -1.77)
 			(end -1.77 -1.77)
@@
 			(layer "F.Fab")
 		)
-		(fp_text user "${REFERENCE}"
-			(at 1.27 2.54 0)
-			(layer "F.Fab")
-			(effects
-				(font
-					(size 1 1)
-					(thickness 0.15)
-				)
-			)
-		)
 		(pad "1" thru_hole rect
 			(at 0 0 90)
@@
 	(footprint "Button_Switch_SMD:SW_Push_1P1T_NO_CK_KMR2"
 		(layer "F.Cu")
-		(at 67.3 96.950001 90)
+		(at 67.3 96.550001 90)
 		(descr "CK components KMR2 tactile switch http://www.ckswitches.com/media/1479/kmr2.pdf")
 		(tags "tactile switch kmr2")
@@
 		(attr smd)
 		(fp_line
-			(start 2.199999 -1.55)
-			(end -2.199999 -1.55)
-			(stroke
-				(width 0.12)
-				(type solid)
-			)
-			(layer "F.SilkS")
-		)
-		(fp_line
 			(start 2.2 0.05)
 			(end 2.2 -0.05)
@@
 		)
 		(fp_line
-			(start -2.199999 1.55)
-			(end 2.199999 1.55)
-			(stroke
-				(width 0.12)
-				(type solid)
-			)
-			(layer "F.SilkS")
-		)
-		(fp_line
 			(start 2.8 -1.8)
 			(end 2.8 1.8)
@@
 	)
 	(gr_line
-		(start 66.85 95.775)
+		(start 66.85 95.8)
 		(end 66.85 95.025)
 		(stroke
@@
 	)
 	(gr_line
-		(start 66.1 95.9)
-		(end 65.6 95.4)
+		(start 66.85 95.8)
+		(end 66.5 95.6)
 		(stroke
 			(width 0.2)
@@
 	)
 	(gr_line
-		(start 74 97.25)
-		(end 73.75 97.5)
+		(start 74 98.875)
+		(end 73.75 99.125)
 		(stroke
 			(width 0.1)
@@
 	)
 	(gr_line
-		(start 67.6 95.9)
-		(end 68.1 95.4)
+		(start 66.85 95.8)
+		(end 67.2 95.6)
 		(stroke
 			(width 0.2)
@@
 	)
 	(gr_line
-		(start 73.75 97.5)
+		(start 73.75 99.125)
 		(end 73.75 103)
 		(stroke
@@
 	)
 	(via
-		(at 68 92.5)
+		(at 70.2 96.6)
 		(size 0.6)
 		(drill 0.3)
@@
 	)
 	(via
-		(at 64.5 95)
+		(at 65 94.6)
 		(size 0.6)
 		(drill 0.3)
@@
 	)
 	(via
-		(at 70.5 95.5)
+		(at 72.8 94.6)
 		(size 0.6)
 		(drill 0.3)
@@
 	)
 	(segment
+		(start 70.6 93.4)
+		(end 73.5 90.5)
+		(width 0.2)
+		(layer "B.Cu")
+		(net 3)
+	)
+	(segment
 		(start 74.5 90.5)
 		(end 78.547 94.547)
@@
 	)
 	(segment
-		(start 62.5 94)
-		(end 70 94)
+		(start 63.1 93.4)
+		(end 70.6 93.4)
 		(width 0.2)
 		(layer "B.Cu")
@@
 	)
 	(segment
-		(start 70 94)
-		(end 73.5 90.5)
+		(start 62.5 94)
+		(end 63.1 93.4)
 		(width 0.2)
 		(layer "B.Cu")
@@
 	)
 	(segment
-		(start 70 99)
-		(end 72.46 101.46)
-		(width 0.2)
-		(layer "F.Cu")
-		(net 12)
-	)
-	(segment
-		(start 72.46 101.46)
-		(end 72.46 101.735)
-		(width 0.2)
-		(layer "F.Cu")
-		(net 12)
-	)
-	(segment
 		(start 68.1 95.9)
 		(end 68.000002 95.999998)
@@
 	)
 	(segment
-		(start 68.1 99)
-		(end 70 99)
+		(start 68.1 98.6)
+		(end 69.6 98.6)
 		(width 0.2)
 		(layer "F.Cu")
@@
 	)
 	(segment
-		(start 68.1 95.9)
-		(end 68.1 94.900002)
+		(start 69.6 98.6)
+		(end 72.46 101.46)
+		(width 0.2)
+		(layer "F.Cu")
+		(net 12)
+	)
+	(segment
+		(start 68.1 94.500002)
+		(end 68.1 98.6)
 		(width 0.2)
 		(layer "F.Cu")
@@
 	)
 	(segment
-		(start 68.1 99)
-		(end 68.1 94.900002)
+		(start 72.46 101.46)
+		(end 72.46 101.735)
 		(width 0.2)
 		(layer "F.Cu")
